File: KiCad/FetsAndCrosses/Gate_NAND3in.sch (KiCad schematic (older format))
At the start: 6 parts, among them Q52 BSS84, Q53 BSS84, Q54 2N7002, Q55 2N7002, Q56 2N7002, Q57 BSS84

Commit message: Schematic Done, Footprints assigned, ERC OK.
Parts:
- Q429: renamed from Q52; footprint (none) -> LogicQ:SOT-23-P
- Q430: renamed from Q53; footprint (none) -> LogicQ:SOT-23-P
- Q431: renamed from Q54; footprint (none) -> LogicQ:SOT-23-N
- Q432: renamed from Q55; footprint (none) -> LogicQ:SOT-23-N
- Q433: renamed from Q56; footprint (none) -> LogicQ:SOT-23-N
- Q434: renamed from Q57; footprint (none) -> LogicQ:SOT-23-P

Commit message: Schematic fixes.
Changed lines of the file:
@@
 $Descr A4 11693 8268
 encoding utf-8
-Sheet 7 389
+Sheet 351 389
 Title ""
-Date ""
-Rev ""
-Comp ""
-Comment1 ""
+Date "2020-07-05"
+Rev "v0.0"
+Comp "Philipp Schilk"
+Comment1 "c"
 Comment2 ""
 Comment3 ""
@@
 AR Path="/5E553405/5F22CC79/5EFE130E/5E56F216" Ref="Q623"  Part="1"
 AR Path="/5E553405/5F22CC79/5EFE130F/5E56F216" Ref="Q629"  Part="1"
-F 0 "Q1301" H 4404 1904 50  0000 L CNN
+F 0 "Q1237" H 4404 1904 50  0000 L CNN
 F 1 "BSS84" H 4404 1995 50  0000 L CNN
 F 2 "LogicQ:SOT-23-P" H 4400 2050 50  0001 C CNN
@@
 AR Path="/5E553405/5F22CC79/5EFE130E/5E570330" Ref="Q624"  Part="1"
 AR Path="/5E553405/5F22CC79/5EFE130F/5E570330" Ref="Q630"  Part="1"
-F 0 "Q1302" H 5354 1904 50  0000 L CNN
+F 0 "Q1238" H 5354 1904 50  0000 L CNN
 F 1 "BSS84" H 5354 1995 50  0000 L CNN
 F 2 "LogicQ:SOT-23-P" H 5350 2050 50  0001 C CNN
@@
 AR Path="/5E553405/5F22CC79/5EFE130E/5E570E83" Ref="Q628"  Part="1"
 AR Path="/5E553405/5F22CC79/5EFE130F/5E570E83" Ref="Q634"  Part="1"
-F 0 "Q1306" H 6304 1904 50  0000 L CNN
+F 0 "Q1242" H 6304 1904 50  0000 L CNN
 F 1 "BSS84" H 6304 1995 50  0000 L CNN
 F 2 "LogicQ:SOT-23-P" H 6300 2050 50  0001 C CNN
@@
 AR Path="/5E553405/5F22CC79/5EFE130E/5E576394" Ref="Q625"  Part="1"
 AR Path="/5E553405/5F22CC79/5EFE130F/5E576394" Ref="Q631"  Part="1"
-F 0 "Q1303" H 5354 3246 50  0000 L CNN
+F 0 "Q1239" H 5354 3246 50  0000 L CNN
 F 1 "2N7002" H 5354 3155 50  0000 L CNN
 F 2 "LogicQ:SOT-23-N" H 5350 3300 50  0001 C CNN
@@
 AR Path="/5E553405/5F22CC79/5EFE130E/5E576894" Ref="Q626"  Part="1"
 AR Path="/5E553405/5F22CC79/5EFE130F/5E576894" Ref="Q632"  Part="1"
-F 0 "Q1304" H 5354 3796 50  0000 L CNN
+F 0 "Q1240" H 5354 3796 50  0000 L CNN
 F 1 "2N7002" H 5354 3705 50  0000 L CNN
 F 2 "LogicQ:SOT-23-N" H 5350 3850 50  0001 C CNN
@@
 AR Path="/5E553405/5F22CC79/5EFE130E/5E57718A" Ref="Q627"  Part="1"
 AR Path="/5E553405/5F22CC79/5EFE130F/5E57718A" Ref="Q633"  Part="1"
-F 0 "Q1305" H 5354 4396 50  0000 L CNN
+F 0 "Q1241" H 5354 4396 50  0000 L CNN
 F 1 "2N7002" H 5354 4305 50  0000 L CNN
 F 2 "LogicQ:SOT-23-N" H 5350 4450 50  0001 C CNN

Commit message: First Draft Schematic Updates
Changed lines of the file:
@@
 $Descr A4 11693 8268
 encoding utf-8
-Sheet 351 389
+Sheet 351 360
 Title ""
 Date "2020-07-05"
@@
 AR Path="/5E553405/5F22CC79/5EFE130E/5E56F216" Ref="Q623"  Part="1"
 AR Path="/5E553405/5F22CC79/5EFE130F/5E56F216" Ref="Q629"  Part="1"
-F 0 "Q1237" H 4404 1904 50  0000 L CNN
+F 0 "Q1301" H 4404 1904 50  0000 L CNN
 F 1 "BSS84" H 4404 1995 50  0000 L CNN
 F 2 "LogicQ:SOT-23-P" H 4400 2050 50  0001 C CNN
@@
 AR Path="/5E553405/5F22CC79/5EFE130E/5E570330" Ref="Q624"  Part="1"
 AR Path="/5E553405/5F22CC79/5EFE130F/5E570330" Ref="Q630"  Part="1"
-F 0 "Q1238" H 5354 1904 50  0000 L CNN
+F 0 "Q1302" H 5354 1904 50  0000 L CNN
 F 1 "BSS84" H 5354 1995 50  0000 L CNN
 F 2 "LogicQ:SOT-23-P" H 5350 2050 50  0001 C CNN
@@
 AR Path="/5E553405/5F22CC79/5EFE130E/5E570E83" Ref="Q628"  Part="1"
 AR Path="/5E553405/5F22CC79/5EFE130F/5E570E83" Ref="Q634"  Part="1"
-F 0 "Q1242" H 6304 1904 50  0000 L CNN
+F 0 "Q1306" H 6304 1904 50  0000 L CNN
 F 1 "BSS84" H 6304 1995 50  0000 L CNN
 F 2 "LogicQ:SOT-23-P" H 6300 2050 50  0001 C CNN
@@
 AR Path="/5E553405/5F22CC79/5EFE130E/5E576394" Ref="Q625"  Part="1"
 AR Path="/5E553405/5F22CC79/5EFE130F/5E576394" Ref="Q631"  Part="1"
-F 0 "Q1239" H 5354 3246 50  0000 L CNN
+F 0 "Q1303" H 5354 3246 50  0000 L CNN
 F 1 "2N7002" H 5354 3155 50  0000 L CNN
 F 2 "LogicQ:SOT-23-N" H 5350 3300 50  0001 C CNN
@@
 AR Path="/5E553405/5F22CC79/5EFE130E/5E576894" Ref="Q626"  Part="1"
 AR Path="/5E553405/5F22CC79/5EFE130F/5E576894" Ref="Q632"  Part="1"
-F 0 "Q1240" H 5354 3796 50  0000 L CNN
+F 0 "Q1304" H 5354 3796 50  0000 L CNN
 F 1 "2N7002" H 5354 3705 50  0000 L CNN
 F 2 "LogicQ:SOT-23-N" H 5350 3850 50  0001 C CNN
@@
 AR Path="/5E553405/5F22CC79/5EFE130E/5E57718A" Ref="Q627"  Part="1"
 AR Path="/5E553405/5F22CC79/5EFE130F/5E57718A" Ref="Q633"  Part="1"
-F 0 "Q1241" H 5354 4396 50  0000 L CNN
+F 0 "Q1305" H 5354 4396 50  0000 L CNN
 F 1 "2N7002" H 5354 4305 50  0000 L CNN
 F 2 "LogicQ:SOT-23-N" H 5350 4450 50  0001 C CNN
