File: KiCad/FetsAndCrosses/Clock.sch (KiCad schematic (older format))
At the start: 0 parts

Commit message: Schematic Done, Footprints assigned, ERC OK.
Parts:
- added C6: 10n, Capacitor_SMD:C_0603_1608Metric, symbol Device:C_Small
- added C7, C8: 0u1, Capacitor_SMD:C_0603_1608Metric, symbol Device:C_Small
- added D97: LED, LogicQ:D_0805_2012Metric_NOLBL, symbol Device:LED_Small
- added Q1362: 2N7002, LogicQ:SOT-23-N, symbol Device:Q_NMOS_GSD
- added R107, R108: 20K, LogicQ:R_0603_1608Metric_NOLBL, symbol Device:R_Small
- added R109: rled, LogicQ:R_0603_1608Metric_NOLBL, symbol Device:R_Small
- added U3: LM555, Package_SO:SO-8_3.9x4.9mm_P1.27mm, symbol Timer:LM555
Connections:
- new net: C8.1, R108.2, U3.2 (TR), U3.6 (THR)
- new net: C6.1, U3.5 (CV)
- new net: R107.1, R108.1, U3.7 (DIS)
- new net: Q1362.3 (D), R109.2
- new net: D97.1 (K), R109.1
- new net +5V: C7.1, D97.2 (A), R107.2, U3.4 (R), U3.8 (VCC)
- new net CLOCK: Q1362.1 (G)
- new net GND: C6.2, C7.2, C8.2, Q1362.2 (S), U3.1 (GND)
- new net sheet5F1B5D77/A: U3.3 (Q)
Other:
- note added: "!"
- note added: "Aprox 240Hz Out"

Commit message: Schematic fixes.
Parts:
- C7, C8: footprint Capacitor_SMD:C_0603_1608Metric -> LogicQ:C_0603_1608Metric_NOLBL
- R107, R108: footprint LogicQ:R_0603_1608Metric_NOLBL -> Resistor_SMD:R_0603_1608Metric
Changed lines of the file:
@@
 Sheet 388 389
 Title ""
-Date ""
-Rev ""
-Comp ""
-Comment1 ""
+Date "2020-07-05"
+Rev "v0.0"
+Comp "Philipp Schilk"
+Comment1 "c"
 Comment2 ""
 Comment3 ""
@@
 F 0 "C7" V 5671 3350 50  0000 C CNN
 F 1 "0u1" V 5762 3350 50  0000 C CNN
-F 2 "Capacitor_SMD:C_0603_1608Metric" H 5900 3350 50  0001 C CNN
+F 2 "LogicQ:C_0603_1608Metric_NOLBL" H 5900 3350 50  0001 C CNN
 F 3 "~" H 5900 3350 50  0001 C CNN
 	1    5900 3350
@@
 F 0 "C8" H 6892 4296 50  0000 L CNN
 F 1 "0u1" H 6892 4205 50  0000 L CNN
-F 2 "Capacitor_SMD:C_0603_1608Metric" H 6800 4250 50  0001 C CNN
+F 2 "LogicQ:C_0603_1608Metric_NOLBL" H 6800 4250 50  0001 C CNN
 F 3 "~" H 6800 4250 50  0001 C CNN
 	1    6800 4250
@@
 F 0 "R108" V 7000 4250 50  0000 C CNN
 F 1 "20K" V 7000 3950 50  0000 C CNN
-F 2 "LogicQ:R_0603_1608Metric_NOLBL" H 7100 4100 50  0001 C CNN
+F 2 "Resistor_SMD:R_0603_1608Metric" H 7100 4100 50  0001 C CNN
 F 3 "~" H 7100 4100 50  0001 C CNN
 	1    7100 4100
@@
 F 0 "R107" V 6550 3550 50  0000 C CNN
 F 1 "20K" V 6550 3250 50  0000 C CNN
-F 2 "LogicQ:R_0603_1608Metric_NOLBL" H 6650 3400 50  0001 C CNN
+F 2 "Resistor_SMD:R_0603_1608Metric" H 6650 3400 50  0001 C CNN
 F 3 "~" H 6650 3400 50  0001 C CNN
 	1    6650 3400

Commit message: First Draft Schematic Updates
Parts:
- removed D97: LED, LogicQ:D_0805_2012Metric_NOLBL, symbol Device:LED_Small
- removed Q1362: 2N7002, LogicQ:SOT-23-N, symbol Device:Q_NMOS_GSD
- removed R109: rled, LogicQ:R_0603_1608Metric_NOLBL, symbol Device:R_Small
Changed lines of the file:
@@
 $Descr A4 11693 8268
 encoding utf-8
-Sheet 388 389
+Sheet 359 360
 Title ""
 Date "2020-07-05"
@@
 $EndComp
 $Comp
-L Device:Q_NMOS_GSD Q?
-U 1 1 5F1B9FA3
-P 8700 5150
-AR Path="/5E53AD22/5E550B0F/5F1B9FA3" Ref="Q?"  Part="1"
-AR Path="/5E53AD22/5E56E0A4/5F1B9FA3" Ref="Q?"  Part="1"
-AR Path="/5E53AD22/5E56E1C0/5F1B9FA3" Ref="Q?"  Part="1"
-AR Path="/5E53AD22/5E56E539/5F1B9FA3" Ref="Q?"  Part="1"
-AR Path="/5E53AD22/5E56E53D/5F1B9FA3" Ref="Q?"  Part="1"
-AR Path="/5E53AD22/5E56E541/5F1B9FA3" Ref="Q?"  Part="1"
-AR Path="/5E53AD22/5E56E941/5F1B9FA3" Ref="Q?"  Part="1"
-AR Path="/5E53AD22/5E56E945/5F1B9FA3" Ref="Q?"  Part="1"
-AR Path="/5E53AD22/5E56E949/5F1B9FA3" Ref="Q?"  Part="1"
-AR Path="/5E53AD22/5E6A228F/5F1B9FA3" Ref="Q?"  Part="1"
-AR Path="/5F18A492/5F1B9FA3" Ref="Q1362"  Part="1"
-F 0 "Q1362" H 8904 5196 50  0000 L CNN
-F 1 "2N7002" H 8904 5105 50  0000 L CNN
-F 2 "LogicQ:SOT-23-N" H 8900 5250 50  0001 C CNN
-F 3 "~" H 8700 5150 50  0001 C CNN
-	1    8700 5150
-	1    0    0    -1
-$EndComp
-$Comp
-L power:GND #PWR?
-U 1 1 5F1B9FA9
-P 8800 5400
-AR Path="/5E53AD22/5E550B0F/5F1B9FA9" Ref="#PWR?"  Part="1"
-AR Path="/5E53AD22/5E56E0A4/5F1B9FA9" Ref="#PWR?"  Part="1"
-AR Path="/5E53AD22/5E56E1C0/5F1B9FA9" Ref="#PWR?"  Part="1"
-AR Path="/5E53AD22/5E56E539/5F1B9FA9" Ref="#PWR?"  Part="1"
-AR Path="/5E53AD22/5E56E53D/5F1B9FA9" Ref="#PWR?"  Part="1"
-AR Path="/5E53AD22/5E56E541/5F1B9FA9" Ref="#PWR?"  Part="1"
-AR Path="/5E53AD22/5E56E941/5F1B9FA9" Ref="#PWR?"  Part="1"
-AR Path="/5E53AD22/5E56E945/5F1B9FA9" Ref="#PWR?"  Part="1"
-AR Path="/5E53AD22/5E56E949/5F1B9FA9" Ref="#PWR?"  Part="1"
-AR Path="/5E53AD22/5E6A228F/5F1B9FA9" Ref="#PWR?"  Part="1"
-AR Path="/5F18A492/5F1B9FA9" Ref="#PWR01093"  Part="1"
-F 0 "#PWR01093" H 8800 5150 50  0001 C CNN
-F 1 "GND" H 8805 5227 50  0000 C CNN
-F 2 "" H 8800 5400 50  0001 C CNN
-F 3 "" H 8800 5400 50  0001 C CNN
-	1    8800 5400
-	1    0    0    -1
-$EndComp
-$Comp
-L Device:LED_Small D?
-U 1 1 5F1B9FB1
-P 8800 4400
-AR Path="/5E53AD22/5E550B0F/5F1B9FB1" Ref="D?"  Part="1"
-AR Path="/5E53AD22/5E56E0A4/5F1B9FB1" Ref="D?"  Part="1"
-AR Path="/5E53AD22/5E56E1C0/5F1B9FB1" Ref="D?"  Part="1"
-AR Path="/5E53AD22/5E56E539/5F1B9FB1" Ref="D?"  Part="1"
-AR Path="/5E53AD22/5E56E53D/5F1B9FB1" Ref="D?"  Part="1"
-AR Path="/5E53AD22/5E56E541/5F1B9FB1" Ref="D?"  Part="1"
-AR Path="/5E53AD22/5E56E941/5F1B9FB1" Ref="D?"  Part="1"
-AR Path="/5E53AD22/5E56E945/5F1B9FB1" Ref="D?"  Part="1"
-AR Path="/5E53AD22/5E56E949/5F1B9FB1" Ref="D?"  Part="1"
-AR Path="/5E53AD22/5E6A228F/5F1B9FB1" Ref="D?"  Part="1"
-AR Path="/5F18A492/5F1B9FB1" Ref="D97"  Part="1"
-F 0 "D97" V 8846 4332 50  0000 R CNN
-F 1 "LED" V 8755 4332 50  0000 R CNN
-F 2 "LogicQ:D_0805_2012Metric_NOLBL" V 8800 4400 50  0001 C CNN
-F 3 "~" V 8800 4400 50  0001 C CNN
-	1    8800 4400
-	0    -1   -1   0
-$EndComp
-$Comp
-L Device:R_Small R?
-U 1 1 5F1B9FB7
-P 8800 4650
-AR Path="/5E53AD22/5E550B0F/5F1B9FB7" Ref="R?"  Part="1"
-AR Path="/5E53AD22/5E56E0A4/5F1B9FB7" Ref="R?"  Part="1"
-AR Path="/5E53AD22/5E56E1C0/5F1B9FB7" Ref="R?"  Part="1"
-AR Path="/5E53AD22/5E56E539/5F1B9FB7" Ref="R?"  Part="1"
-AR Path="/5E53AD22/5E56E53D/5F1B9FB7" Ref="R?"  Part="1"
-AR Path="/5E53AD22/5E56E541/5F1B9FB7" Ref="R?"  Part="1"
-AR Path="/5E53AD22/5E56E941/5F1B9FB7" Ref="R?"  Part="1"
-AR Path="/5E53AD22/5E56E945/5F1B9FB7" Ref="R?"  Part="1"
-AR Path="/5E53AD22/5E56E949/5F1B9FB7" Ref="R?"  Part="1"
-AR Path="/5E53AD22/5E6A228F/5F1B9FB7" Ref="R?"  Part="1"
-AR Path="/5F18A492/5F1B9FB7" Ref="R109"  Part="1"
-F 0 "R109" H 8859 4696 50  0000 L CNN
-F 1 "rled" H 8859 4605 50  0000 L CNN
-F 2 "LogicQ:R_0603_1608Metric_NOLBL" H 8800 4650 50  0001 C CNN
-F 3 "~" H 8800 4650 50  0001 C CNN
-	1    8800 4650
-	1    0    0    -1
-$EndComp
-$Comp
-L power:+5V #PWR01094
-U 1 1 5F1BC956
-P 8800 4200
-F 0 "#PWR01094" H 8800 4050 50  0001 C CNN
-F 1 "+5V" H 8815 4373 50  0000 C CNN
-F 2 "" H 8800 4200 50  0001 C CNN
-F 3 "" H 8800 4200 50  0001 C CNN
-	1    8800 4200
-	1    0    0    -1
-$EndComp
-$Comp
 L Device:C_Small C8
 U 1 1 5F1C0AA1
@@
 	5100 4400 5100 4350
 Wire Wire Line
-	8800 5400 8800 5350
-Wire Wire Line
-	8800 4550 8800 4500
-Wire Wire Line
-	8800 4750 8800 4950
-Wire Wire Line
-	8800 4200 8800 4300
-Wire Wire Line
-	8100 3700 8100 5150
-Wire Wire Line
-	8100 5150 8500 5150
-Wire Wire Line
-	8100 3700 8450 3700
-Wire Wire Line
 	5550 3700 5050 3700
 Wire Wire Line
@@
 Wire Wire Line
 	6650 3200 6650 3300
-Wire Wire Line
-	8100 3700 7950 3700
 Wire Wire Line
 	6550 3700 7400 3700
@@
 Connection ~ 6800 4100
 Connection ~ 6650 3900
-Connection ~ 8100 3700
+Wire Wire Line
+	7950 3700 8450 3700
 $EndSCHEMATC

Commit message: PCB v1.0 layout mostly done.
Parts:
- U3: symbol Timer:LM555 -> FetsAndCrosses-rescue:LM555-Timer
Changed lines of the file:
@@
 $EndSheet
 $Comp
-L Timer:LM555 U3
+L FetsAndCrosses-rescue:LM555-Timer U3
 U 1 1 5F1ABDD6
 P 6050 3900
+AR Path="/5F1ABDD6" Ref="U3"  Part="1"
+AR Path="/5F18A492/5F1ABDD6" Ref="U3"  Part="1"
 F 0 "U3" H 6200 4350 50  0000 C CNN
 F 1 "LM555" H 6250 4250 50  0000 C CNN
