File: KiCad/Engine/Cell1in.sch (KiCad schematic (older format))
At the start: 0 parts

Commit message: Engine Fixes
Changed lines of the file:
@@
 $Descr A4 11693 8268
 encoding utf-8
-Sheet 350 398
+Sheet 137 398
 Title ""
 Date ""
@@
 	6450 2300 6450 2650
 Text HLabel 5150 2750 0    50   Input ~ 0
-Inhib
+Block
 Text HLabel 7850 2700 2    50   Output ~ 0
-Inhib_Out
+Block_Out
 $Sheet
 S 5400 2150 550  300
