File: KiCad/Engine/Engine_EMPTY_SIDES.sch (KiCad schematic (older format))
At the start: 0 parts

Commit message: Engine Fixes
Changed lines of the file:
@@
 $Descr A4 11693 8268
 encoding utf-8
-Sheet 344 398
+Sheet 119 398
 Title ""
 Date ""
@@
 F2 "A" I L 4050 2150 50
 F3 "Out" O R 4850 2150 50
-F4 "Inhib" I L 4050 2050 50
-F5 "Inhib_Out" O R 4850 2050 50
+F4 "Block" I L 4050 2050 50
+F5 "Block_Out" O R 4850 2050 50
 $EndSheet
 $Sheet
@@
 F2 "A" I L 8050 2150 50
 F3 "Out" O R 8850 2150 50
-F4 "Inhib" I L 8050 2050 50
-F5 "Inhib_Out" O R 8850 2050 50
+F4 "Block" I L 8050 2050 50
+F5 "Block_Out" O R 8850 2050 50
 $EndSheet
 Wire Wire Line
@@
 F2 "A" I L 6050 2150 50
 F3 "Out" O R 6850 2150 50
-F4 "Inhib" I L 6050 2050 50
-F5 "Inhib_Out" O R 6850 2050 50
+F4 "Block" I L 6050 2050 50
+F5 "Block_Out" O R 6850 2050 50
 $EndSheet
 Wire Wire Line

Commit message: Engine layout.
Connections:
- net labels added: Block
- net labels removed: Inhib
Changed lines of the file:
@@
 $Descr A4 11693 8268
 encoding utf-8
-Sheet 119 398
+Sheet 382 398
 Title ""
 Date ""
@@
 	4050 2050 3700 2050
 Text HLabel 3700 2050 0    50   Input ~ 0
-Inhib
+Block
 Wire Wire Line
 	9650 2800 9650 2050
