File: ECAD/Engine/KiCad/Gate_NOR3in.sch (KiCad schematic (older format))
At the start: 6 parts, among them Q421 2N7002, Q422 2N7002, Q423 BSS84, Q424 BSS84, Q425 BSS84, Q426 2N7002

Commit message: Engine: Added Tooling Holes, LCSC Part numbers
Parts:
- Q421, Q422, Q426: LCSC (none) -> C8545
- Q423, Q424, Q425: LCSC (none) -> C114481
Changed lines of the file:
@@
 F 2 "LogicQ:SOT-23-P" H 6000 2950 50  0001 C CNN
 F 3 "~" H 5800 2850 50  0001 C CNN
+F 4 "C114481" H 5800 2850 50  0001 C CNN "LCSC"
 	1    5800 2850
 	1    0    0    1
@@
 F 2 "LogicQ:SOT-23-N" H 5500 4700 50  0001 C CNN
 F 3 "~" H 5300 4600 50  0001 C CNN
+F 4 "C8545" H 5300 4600 50  0001 C CNN "LCSC"
 	1    5300 4600
 	1    0    0    -1
@@
 F 2 "LogicQ:SOT-23-P" H 6000 2300 50  0001 C CNN
 F 3 "~" H 5800 2200 50  0001 C CNN
+F 4 "C114481" H 5800 2200 50  0001 C CNN "LCSC"
 	1    5800 2200
 	1    0    0    1
@@
 F 2 "LogicQ:SOT-23-N" H 6450 4700 50  0001 C CNN
 F 3 "~" H 6250 4600 50  0001 C CNN
+F 4 "C8545" H 6250 4600 50  0001 C CNN "LCSC"
 	1    6250 4600
 	1    0    0    -1
@@
 F 2 "LogicQ:SOT-23-P" H 6000 3700 50  0001 C CNN
 F 3 "~" H 5800 3600 50  0001 C CNN
+F 4 "C114481" H 5800 3600 50  0001 C CNN "LCSC"
 	1    5800 3600
 	1    0    0    1
@@
 F 2 "LogicQ:SOT-23-N" H 4550 4700 50  0001 C CNN
 F 3 "~" H 4350 4600 50  0001 C CNN
+F 4 "C8545" H 4350 4600 50  0001 C CNN "LCSC"
 	1    4350 4600
 	1    0    0    -1
