File: ECAD/Engine/KiCad/Gate_NOR8in.sch (KiCad schematic (older format))
At the start: 16 parts, among them Q1346 BSS84, Q1347 BSS84, Q1348 2N7002, Q1349 2N7002, Q1350 BSS84, Q1351 BSS84, Q1352 BSS84, Q1353 2N7002, Q1354 2N7002, Q1355 2N7002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

Commit message: Engine: Added Tooling Holes, LCSC Part numbers
Parts:
- Q1346, Q1347, Q1350, Q1351, Q1352, Q1356, Q1357, Q1358: LCSC (none) -> C114481
- Q1348, Q1349, Q1353, Q1354, Q1355, Q1359, Q1360, Q1361: LCSC (none) -> C8545
Changed lines of the file:
@@
 F 2 "LogicQ:SOT-23-P" H 4300 2600 50  0001 C CNN
 F 3 "~" H 4100 2500 50  0001 C CNN
+F 4 "C114481" H 4100 2500 50  0001 C CNN "LCSC"
 	1    4100 2500
 	1    0    0    1
@@
 F 2 "LogicQ:SOT-23-N" H 7300 3550 50  0001 C CNN
 F 3 "~" H 7100 3450 50  0001 C CNN
+F 4 "C8545" H 7100 3450 50  0001 C CNN "LCSC"
 	1    7100 3450
 	1    0    0    -1
@@
 F 2 "LogicQ:SOT-23-P" H 4300 2100 50  0001 C CNN
 F 3 "~" H 4100 2000 50  0001 C CNN
+F 4 "C114481" H 4100 2000 50  0001 C CNN "LCSC"
 	1    4100 2000
 	1    0    0    1
@@
 F 2 "LogicQ:SOT-23-P" H 5750 2100 50  0001 C CNN
 F 3 "~" H 5550 2000 50  0001 C CNN
+F 4 "C114481" H 5550 2000 50  0001 C CNN "LCSC"
 	1    5550 2000
 	1    0    0    1
@@
 F 2 "LogicQ:SOT-23-P" H 5750 1600 50  0001 C CNN
 F 3 "~" H 5550 1500 50  0001 C CNN
+F 4 "C114481" H 5550 1500 50  0001 C CNN "LCSC"
 	1    5550 1500
 	1    0    0    1
@@
 F 2 "LogicQ:SOT-23-P" H 7300 2600 50  0001 C CNN
 F 3 "~" H 7100 2500 50  0001 C CNN
+F 4 "C114481" H 7100 2500 50  0001 C CNN "LCSC"
 	1    7100 2500
 	1    0    0    1
@@
 F 2 "LogicQ:SOT-23-P" H 7300 2100 50  0001 C CNN
 F 3 "~" H 7100 2000 50  0001 C CNN
+F 4 "C114481" H 7100 2000 50  0001 C CNN "LCSC"
 	1    7100 2000
 	1    0    0    1
@@
 F 2 "LogicQ:SOT-23-P" H 7300 1600 50  0001 C CNN
 F 3 "~" H 7100 1500 50  0001 C CNN
+F 4 "C114481" H 7100 1500 50  0001 C CNN "LCSC"
 	1    7100 1500
 	1    0    0    1
@@
 F 2 "LogicQ:SOT-23-N" H 5750 3550 50  0001 C CNN
 F 3 "~" H 5550 3450 50  0001 C CNN
+F 4 "C8545" H 5550 3450 50  0001 C CNN "LCSC"
 	1    5550 3450
 	1    0    0    -1
@@
 F 2 "LogicQ:SOT-23-N" H 7300 4450 50  0001 C CNN
 F 3 "~" H 7100 4350 50  0001 C CNN
+F 4 "C8545" H 7100 4350 50  0001 C CNN "LCSC"
 	1    7100 4350
 	1    0    0    -1
@@
 F 2 "LogicQ:SOT-23-N" H 5750 4450 50  0001 C CNN
 F 3 "~" H 5550 4350 50  0001 C CNN
+F 4 "C8545" H 5550 4350 50  0001 C CNN "LCSC"
 	1    5550 4350
 	1    0    0    -1
@@
 F 2 "LogicQ:SOT-23-N" H 4300 4450 50  0001 C CNN
 F 3 "~" H 4100 4350 50  0001 C CNN
+F 4 "C8545" H 4100 4350 50  0001 C CNN "LCSC"
 	1    4100 4350
 	1    0    0    -1
@@
 F 2 "LogicQ:SOT-23-N" H 7300 5350 50  0001 C CNN
 F 3 "~" H 7100 5250 50  0001 C CNN
+F 4 "C8545" H 7100 5250 50  0001 C CNN "LCSC"
 	1    7100 5250
 	1    0    0    -1
@@
 F 2 "LogicQ:SOT-23-N" H 5750 5350 50  0001 C CNN
 F 3 "~" H 5550 5250 50  0001 C CNN
+F 4 "C8545" H 5550 5250 50  0001 C CNN "LCSC"
 	1    5550 5250
 	1    0    0    -1
@@
 F 2 "LogicQ:SOT-23-N" H 4300 5350 50  0001 C CNN
 F 3 "~" H 4100 5250 50  0001 C CNN
+F 4 "C8545" H 4100 5250 50  0001 C CNN "LCSC"
 	1    4100 5250
 	1    0    0    -1
@@
 F 2 "LogicQ:SOT-23-P" H 5750 2600 50  0001 C CNN
 F 3 "~" H 5550 2500 50  0001 C CNN
+F 4 "C114481" H 5550 2500 50  0001 C CNN "LCSC"
 	1    5550 2500
 	1    0    0    1
