File: ECAD/Fets_and_Crosses/KiCad/Gate_NAND2in.sch (KiCad schematic (older format))
At the start: 4 parts, among them Q771 BSS84, Q772 2N7002, Q773 2N7002, Q774 BSS84

Commit message: Added Most LCSC Part Numbers
Parts:
- Q771, Q774: LCSC (none) -> C114481
- Q772, Q773: LCSC (none) -> C8545
Changed lines of the file:
@@
 F 2 "LogicQ:SOT-23-P" H 6450 3050 50  0001 C CNN
 F 3 "~" H 6250 2950 50  0001 C CNN
+F 4 "C114481" H 6250 2950 50  0001 C CNN "LCSC"
 	1    6250 2950
 	1    0    0    1
@@
 F 2 "LogicQ:SOT-23-N" H 6800 3750 50  0001 C CNN
 F 3 "~" H 6600 3650 50  0001 C CNN
+F 4 "C8545" H 6600 3650 50  0001 C CNN "LCSC"
 	1    6600 3650
 	1    0    0    -1
@@
 F 2 "LogicQ:SOT-23-P" H 7250 3050 50  0001 C CNN
 F 3 "~" H 7050 2950 50  0001 C CNN
+F 4 "C114481" H 7050 2950 50  0001 C CNN "LCSC"
 	1    7050 2950
 	1    0    0    1
@@
 F 2 "LogicQ:SOT-23-N" H 6800 4450 50  0001 C CNN
 F 3 "~" H 6600 4350 50  0001 C CNN
+F 4 "C8545" H 6600 4350 50  0001 C CNN "LCSC"
 	1    6600 4350
 	1    0    0    -1
