File: ECAD/Fets_and_Crosses/KiCad/Gate_NAND3in.sch (KiCad schematic (older format))
At the start: 6 parts, among them Q429 BSS84, Q430 BSS84, Q431 2N7002, Q432 2N7002, Q433 2N7002, Q434 BSS84

Commit message: Cleanup
Changed lines of the file:
@@
 $Descr A4 11693 8268
 encoding utf-8
-Sheet 316 362
+Sheet 341 362
 Title "Fets and Crosses"
 Date "2021-05-23"
@@
 AR Path="/5E553405/5F22CC79/5EFE130E/5E56F216" Ref="Q623"  Part="1"
 AR Path="/5E553405/5F22CC79/5EFE130F/5E56F216" Ref="Q629"  Part="1"
-F 0 "Q1301" H 4404 1904 50  0000 L CNN
+F 0 "Q1295" H 4404 1904 50  0000 L CNN
 F 1 "BSS84" H 4404 1995 50  0000 L CNN
 F 2 "LogicQ:SOT-23-P" H 4400 2050 50  0001 C CNN
@@
 AR Path="/5E553405/5F22CC79/5EFE130E/5E570330" Ref="Q624"  Part="1"
 AR Path="/5E553405/5F22CC79/5EFE130F/5E570330" Ref="Q630"  Part="1"
-F 0 "Q1302" H 5354 1904 50  0000 L CNN
+F 0 "Q1296" H 5354 1904 50  0000 L CNN
 F 1 "BSS84" H 5354 1995 50  0000 L CNN
 F 2 "LogicQ:SOT-23-P" H 5350 2050 50  0001 C CNN
@@
 AR Path="/5E553405/5F22CC79/5EFE130E/5E570E83" Ref="Q628"  Part="1"
 AR Path="/5E553405/5F22CC79/5EFE130F/5E570E83" Ref="Q634"  Part="1"
-F 0 "Q1306" H 6304 1904 50  0000 L CNN
+F 0 "Q1300" H 6304 1904 50  0000 L CNN
 F 1 "BSS84" H 6304 1995 50  0000 L CNN
 F 2 "LogicQ:SOT-23-P" H 6300 2050 50  0001 C CNN
@@
 AR Path="/5E553405/5F22CC79/5EFE130E/5E576394" Ref="Q625"  Part="1"
 AR Path="/5E553405/5F22CC79/5EFE130F/5E576394" Ref="Q631"  Part="1"
-F 0 "Q1303" H 5354 3246 50  0000 L CNN
+F 0 "Q1297" H 5354 3246 50  0000 L CNN
 F 1 "2N7002" H 5354 3155 50  0000 L CNN
 F 2 "LogicQ:SOT-23-N" H 5350 3300 50  0001 C CNN
@@
 AR Path="/5E553405/5F22CC79/5EFE130E/5E576894" Ref="Q626"  Part="1"
 AR Path="/5E553405/5F22CC79/5EFE130F/5E576894" Ref="Q632"  Part="1"
-F 0 "Q1304" H 5354 3796 50  0000 L CNN
+F 0 "Q1298" H 5354 3796 50  0000 L CNN
 F 1 "2N7002" H 5354 3705 50  0000 L CNN
 F 2 "LogicQ:SOT-23-N" H 5350 3850 50  0001 C CNN
@@
 AR Path="/5E553405/5F22CC79/5EFE130E/5E57718A" Ref="Q627"  Part="1"
 AR Path="/5E553405/5F22CC79/5EFE130F/5E57718A" Ref="Q633"  Part="1"
-F 0 "Q1305" H 5354 4396 50  0000 L CNN
+F 0 "Q1299" H 5354 4396 50  0000 L CNN
 F 1 "2N7002" H 5354 4305 50  0000 L CNN
 F 2 "LogicQ:SOT-23-N" H 5350 4450 50  0001 C CNN

Commit message: POR, Tooling Holes
Changed lines of the file:
@@
 $Descr A4 11693 8268
 encoding utf-8
-Sheet 341 362
+Sheet 341 363
 Title "Fets and Crosses"
 Date "2021-05-23"
@@
 AR Path="/5E553405/5F22CC79/5EFE130E/5E56F216" Ref="Q623"  Part="1"
 AR Path="/5E553405/5F22CC79/5EFE130F/5E56F216" Ref="Q629"  Part="1"
-F 0 "Q1295" H 4404 1904 50  0000 L CNN
+F 0 "Q1301" H 4404 1904 50  0000 L CNN
 F 1 "BSS84" H 4404 1995 50  0000 L CNN
 F 2 "LogicQ:SOT-23-P" H 4400 2050 50  0001 C CNN
@@
 AR Path="/5E553405/5F22CC79/5EFE130E/5E570330" Ref="Q624"  Part="1"
 AR Path="/5E553405/5F22CC79/5EFE130F/5E570330" Ref="Q630"  Part="1"
-F 0 "Q1296" H 5354 1904 50  0000 L CNN
+F 0 "Q1302" H 5354 1904 50  0000 L CNN
 F 1 "BSS84" H 5354 1995 50  0000 L CNN
 F 2 "LogicQ:SOT-23-P" H 5350 2050 50  0001 C CNN
@@
 AR Path="/5E553405/5F22CC79/5EFE130E/5E570E83" Ref="Q628"  Part="1"
 AR Path="/5E553405/5F22CC79/5EFE130F/5E570E83" Ref="Q634"  Part="1"
-F 0 "Q1300" H 6304 1904 50  0000 L CNN
+F 0 "Q1306" H 6304 1904 50  0000 L CNN
 F 1 "BSS84" H 6304 1995 50  0000 L CNN
 F 2 "LogicQ:SOT-23-P" H 6300 2050 50  0001 C CNN
@@
 AR Path="/5E553405/5F22CC79/5EFE130E/5E576394" Ref="Q625"  Part="1"
 AR Path="/5E553405/5F22CC79/5EFE130F/5E576394" Ref="Q631"  Part="1"
-F 0 "Q1297" H 5354 3246 50  0000 L CNN
+F 0 "Q1303" H 5354 3246 50  0000 L CNN
 F 1 "2N7002" H 5354 3155 50  0000 L CNN
 F 2 "LogicQ:SOT-23-N" H 5350 3300 50  0001 C CNN
@@
 AR Path="/5E553405/5F22CC79/5EFE130E/5E576894" Ref="Q626"  Part="1"
 AR Path="/5E553405/5F22CC79/5EFE130F/5E576894" Ref="Q632"  Part="1"
-F 0 "Q1298" H 5354 3796 50  0000 L CNN
+F 0 "Q1304" H 5354 3796 50  0000 L CNN
 F 1 "2N7002" H 5354 3705 50  0000 L CNN
 F 2 "LogicQ:SOT-23-N" H 5350 3850 50  0001 C CNN
@@
 AR Path="/5E553405/5F22CC79/5EFE130E/5E57718A" Ref="Q627"  Part="1"
 AR Path="/5E553405/5F22CC79/5EFE130F/5E57718A" Ref="Q633"  Part="1"
-F 0 "Q1299" H 5354 4396 50  0000 L CNN
+F 0 "Q1305" H 5354 4396 50  0000 L CNN
 F 1 "2N7002" H 5354 4305 50  0000 L CNN
 F 2 "LogicQ:SOT-23-N" H 5350 4450 50  0001 C CNN

Commit message: Added Most LCSC Part Numbers
Parts:
- Q429, Q430, Q434: LCSC (none) -> C114481
- Q431, Q432, Q433: LCSC (none) -> C8545
Changed lines of the file:
@@
 F 2 "LogicQ:SOT-23-P" H 4400 2050 50  0001 C CNN
 F 3 "~" H 4200 1950 50  0001 C CNN
+F 4 "C114481" H 4200 1950 50  0001 C CNN "LCSC"
 	1    4200 1950
 	1    0    0    1
@@
 F 2 "LogicQ:SOT-23-P" H 5350 2050 50  0001 C CNN
 F 3 "~" H 5150 1950 50  0001 C CNN
+F 4 "C114481" H 5150 1950 50  0001 C CNN "LCSC"
 	1    5150 1950
 	1    0    0    1
@@
 F 2 "LogicQ:SOT-23-P" H 6300 2050 50  0001 C CNN
 F 3 "~" H 6100 1950 50  0001 C CNN
+F 4 "C114481" H 6100 1950 50  0001 C CNN "LCSC"
 	1    6100 1950
 	1    0    0    1
@@
 F 2 "LogicQ:SOT-23-N" H 5350 3300 50  0001 C CNN
 F 3 "~" H 5150 3200 50  0001 C CNN
+F 4 "C8545" H 5150 3200 50  0001 C CNN "LCSC"
 	1    5150 3200
 	1    0    0    -1
@@
 F 2 "LogicQ:SOT-23-N" H 5350 3850 50  0001 C CNN
 F 3 "~" H 5150 3750 50  0001 C CNN
+F 4 "C8545" H 5150 3750 50  0001 C CNN "LCSC"
 	1    5150 3750
 	1    0    0    -1
@@
 F 2 "LogicQ:SOT-23-N" H 5350 4450 50  0001 C CNN
 F 3 "~" H 5150 4350 50  0001 C CNN
+F 4 "C8545" H 5150 4350 50  0001 C CNN "LCSC"
 	1    5150 4350
 	1    0    0    -1
