File: ECAD/Fets_and_Crosses/KiCad/Gate_NAND8in.sch (KiCad schematic (older format))
At the start: 16 parts, among them Q477 BSS84, Q478 BSS84, Q479 2N7002, Q480 2N7002, Q481 BSS84, Q482 BSS84, Q483 BSS84, Q484 2N7002, Q485 2N7002, Q486 2N7002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

Commit message: Added Most LCSC Part Numbers
Parts:
- Q477, Q478, Q481, Q482, Q483, Q487, Q488, Q489: LCSC (none) -> C114481
- Q479, Q480, Q484, Q485, Q486, Q490, Q491, Q492: LCSC (none) -> C8545
Changed lines of the file:
@@
 F 2 "LogicQ:SOT-23-P" H 5050 1750 50  0001 C CNN
 F 3 "~" H 4850 1650 50  0001 C CNN
+F 4 "C114481" H 4850 1650 50  0001 C CNN "LCSC"
 	1    4850 1650
 	1    0    0    1
@@
 F 2 "LogicQ:SOT-23-P" H 6600 1750 50  0001 C CNN
 F 3 "~" H 6400 1650 50  0001 C CNN
+F 4 "C114481" H 6400 1650 50  0001 C CNN "LCSC"
 	1    6400 1650
 	1    0    0    1
@@
 F 2 "LogicQ:SOT-23-P" H 6600 2650 50  0001 C CNN
 F 3 "~" H 6400 2550 50  0001 C CNN
+F 4 "C114481" H 6400 2550 50  0001 C CNN "LCSC"
 	1    6400 2550
 	1    0    0    1
@@
 F 2 "LogicQ:SOT-23-P" H 5050 2650 50  0001 C CNN
 F 3 "~" H 4850 2550 50  0001 C CNN
+F 4 "C114481" H 4850 2550 50  0001 C CNN "LCSC"
 	1    4850 2550
 	1    0    0    1
@@
 F 2 "LogicQ:SOT-23-P" H 6600 3550 50  0001 C CNN
 F 3 "~" H 6400 3450 50  0001 C CNN
+F 4 "C114481" H 6400 3450 50  0001 C CNN "LCSC"
 	1    6400 3450
 	1    0    0    1
@@
 F 2 "LogicQ:SOT-23-P" H 5050 3550 50  0001 C CNN
 F 3 "~" H 4850 3450 50  0001 C CNN
+F 4 "C114481" H 4850 3450 50  0001 C CNN "LCSC"
 	1    4850 3450
 	1    0    0    1
@@
 F 2 "LogicQ:SOT-23-P" H 3600 3550 50  0001 C CNN
 F 3 "~" H 3400 3450 50  0001 C CNN
+F 4 "C114481" H 3400 3450 50  0001 C CNN "LCSC"
 	1    3400 3450
 	1    0    0    1
@@
 F 2 "LogicQ:SOT-23-N" H 3600 5300 50  0001 C CNN
 F 3 "~" H 3400 5200 50  0001 C CNN
+F 4 "C8545" H 3400 5200 50  0001 C CNN "LCSC"
 	1    3400 5200
 	1    0    0    -1
@@
 F 2 "LogicQ:SOT-23-N" H 3600 5800 50  0001 C CNN
 F 3 "~" H 3400 5700 50  0001 C CNN
+F 4 "C8545" H 3400 5700 50  0001 C CNN "LCSC"
 	1    3400 5700
 	1    0    0    -1
@@
 F 2 "LogicQ:SOT-23-N" H 5050 5800 50  0001 C CNN
 F 3 "~" H 4850 5700 50  0001 C CNN
+F 4 "C8545" H 4850 5700 50  0001 C CNN "LCSC"
 	1    4850 5700
 	1    0    0    -1
@@
 F 2 "LogicQ:SOT-23-N" H 5050 5300 50  0001 C CNN
 F 3 "~" H 4850 5200 50  0001 C CNN
+F 4 "C8545" H 4850 5200 50  0001 C CNN "LCSC"
 	1    4850 5200
 	1    0    0    -1
@@
 F 2 "LogicQ:SOT-23-N" H 5050 4800 50  0001 C CNN
 F 3 "~" H 4850 4700 50  0001 C CNN
+F 4 "C8545" H 4850 4700 50  0001 C CNN "LCSC"
 	1    4850 4700
 	1    0    0    -1
@@
 F 2 "LogicQ:SOT-23-N" H 6600 4800 50  0001 C CNN
 F 3 "~" H 6400 4700 50  0001 C CNN
+F 4 "C8545" H 6400 4700 50  0001 C CNN "LCSC"
 	1    6400 4700
 	1    0    0    -1
@@
 F 2 "LogicQ:SOT-23-N" H 6600 5300 50  0001 C CNN
 F 3 "~" H 6400 5200 50  0001 C CNN
+F 4 "C8545" H 6400 5200 50  0001 C CNN "LCSC"
 	1    6400 5200
 	1    0    0    -1
@@
 F 2 "LogicQ:SOT-23-N" H 6600 5800 50  0001 C CNN
 F 3 "~" H 6400 5700 50  0001 C CNN
+F 4 "C8545" H 6400 5700 50  0001 C CNN "LCSC"
 	1    6400 5700
 	1    0    0    -1
@@
 F 2 "LogicQ:SOT-23-P" H 3600 2650 50  0001 C CNN
 F 3 "~" H 3400 2550 50  0001 C CNN
+F 4 "C114481" H 3400 2550 50  0001 C CNN "LCSC"
 	1    3400 2550
 	1    0    0    1
