File: ECAD/Fets_and_Crosses/KiCad/Gate_SchmittInv.sch (KiCad schematic (older format))
At the start: 6 parts, among them Q1391 BSS84, Q1392 BSS84, Q1393 2N7002, Q1394 2N7002, Q1395 BSS84, Q1396 2N7002

Commit message: Added Most LCSC Part Numbers
Parts:
- Q1391, Q1392, Q1395: LCSC (none) -> C114481
- Q1393, Q1394, Q1396: LCSC (none) -> C8545
Changed lines of the file:
@@
 F 2 "LogicQ:SOT-23-P" H 5200 2750 50  0001 C CNN
 F 3 "~" H 5000 2650 50  0001 C CNN
+F 4 "C114481" H 5000 2650 50  0001 C CNN "LCSC"
 	1    5000 2650
 	1    0    0    1
@@
 F 2 "LogicQ:SOT-23-N" H 5200 3550 50  0001 C CNN
 F 3 "~" H 5000 3450 50  0001 C CNN
+F 4 "C8545" H 5000 3450 50  0001 C CNN "LCSC"
 	1    5000 3450
 	1    0    0    -1
@@
 F 2 "LogicQ:SOT-23-P" H 5200 2050 50  0001 C CNN
 F 3 "~" H 5000 1950 50  0001 C CNN
+F 4 "C114481" H 5000 1950 50  0001 C CNN "LCSC"
 	1    5000 1950
 	1    0    0    1
@@
 F 2 "LogicQ:SOT-23-N" H 5200 4250 50  0001 C CNN
 F 3 "~" H 5000 4150 50  0001 C CNN
+F 4 "C8545" H 5000 4150 50  0001 C CNN "LCSC"
 	1    5000 4150
 	1    0    0    -1
@@
 F 2 "LogicQ:SOT-23-P" H 5900 2500 50  0001 C CNN
 F 3 "~" H 5700 2400 50  0001 C CNN
+F 4 "C114481" H 5700 2400 50  0001 C CNN "LCSC"
 	1    5700 2400
 	0    1    -1   0
@@
 F 2 "LogicQ:SOT-23-N" H 5900 3800 50  0001 C CNN
 F 3 "~" H 5700 3700 50  0001 C CNN
+F 4 "C8545" H 5700 3700 50  0001 C CNN "LCSC"
 	1    5700 3700
 	0    1    1    0
